Commit message: feat: add XACRO model for custom rover with Pixhawk and sensor configuration

File: urdf/pixhawk.urdf.xacro (robot description, xacro)
@@ -92,5 +92,5 @@
       <origin xyz="0 0 0" rpy="0 0 0"/>
       <geometry>
-        <box size="0.056 0.085 0.016"/>
+        <box size="0.082 0.050 0.016"/>
       </geometry>
       <material name="dark_grey"/>
@@ -100,7 +100,7 @@
     <parent link="top_plate"/>
     <child link="pixhawk_link"/>
-    <origin xyz="0.03 0 0.0105" rpy="0 0 0"/>
+    <origin xyz="0.03 0 0.0335" rpy="0 0 0"/>
   </joint>
-  <link name="laser">
+  <link name="laser_frame">
     <visual>
       <origin xyz="0 0 0" rpy="0 0 0"/>
@@ -113,5 +113,5 @@
   <joint name="lidar_joint" type="fixed">
     <parent link="base_link"/>
-    <child link="laser"/>
+    <child link="laser_frame"/>
     <origin xyz="-0.08 0 0.08" rpy="0 0 0"/>
   </joint>

Commit message: feat: add robot URDF model and central bringup launch file for rover hardware components

File: urdf/pixhawk.urdf.xacro (robot description, xacro)
@@ -102,5 +102,19 @@
     <origin xyz="0.03 0 0.0335" rpy="0 0 0"/>
   </joint>
-  <link name="laser_frame">
+  <link name="imu_link">
+    <visual>
+      <origin xyz="0 0 0" rpy="0 0 0"/>
+      <geometry>
+        <box size="0.02 0.015 0.003"/>
+      </geometry>
+      <material name="blue"/>
+    </visual>
+  </link>
+  <joint name="imu_joint" type="fixed">
+    <parent link="top_plate"/>
+    <child link="imu_link"/>
+    <origin xyz="0.04 -0.04 0.004" rpy="0 0 0"/>
+  </joint>
+  <link name="laser">
     <visual>
       <origin xyz="0 0 0" rpy="0 0 0"/>
@@ -113,5 +127,5 @@
   <joint name="lidar_joint" type="fixed">
     <parent link="base_link"/>
-    <child link="laser_frame"/>
+    <child link="laser"/>
     <origin xyz="-0.08 0 0.08" rpy="0 0 0"/>
   </joint>
