Commit message: fix(urdf): set wheel separation to 0.28m and wheel radius to 0.050m

File: urdf/BNO055.urdf.xacro (robot description, xacro)
@@ -118,5 +118,5 @@
         <origin xyz="0 0 0" rpy="${pi/2} 0 0"/>
         <geometry>
-          <cylinder radius="0.045" length="0.03"/>
+          <cylinder radius="0.050" length="0.03"/>
         </geometry>
         <material name="black"/>
@@ -125,5 +125,5 @@
         <origin xyz="0 0 0" rpy="${pi/2} 0 0"/>
         <geometry>
-          <cylinder radius="0.045" length="0.03"/>
+          <cylinder radius="0.050" length="0.03"/>
         </geometry>
       </collision>
@@ -132,5 +132,5 @@
       <parent link="base_link"/>
       <child link="${prefix}_wheel"/>
-      <origin xyz="${x_reflect * 0.115} ${y_reflect * 0.115} -0.015" rpy="0 0 0"/>
+      <origin xyz="${x_reflect * 0.115} ${y_reflect * 0.140} -0.015" rpy="0 0 0"/>
       <axis xyz="0 1 0"/>
     </joint>

File: urdf/pixhawk.urdf.xacro (robot description, xacro)
@@ -121,5 +121,5 @@
         <origin xyz="0 0 0" rpy="${pi/2} 0 0"/>
         <geometry>
-          <cylinder radius="0.045" length="0.03"/>
+          <cylinder radius="0.050" length="0.03"/>
         </geometry>
         <material name="black"/>
@@ -128,5 +128,5 @@
         <origin xyz="0 0 0" rpy="${pi/2} 0 0"/>
         <geometry>
-          <cylinder radius="0.045" length="0.03"/>
+          <cylinder radius="0.050" length="0.03"/>
         </geometry>
       </collision>
@@ -135,5 +135,5 @@
       <parent link="base_link"/>
       <child link="${prefix}_wheel"/>
-      <origin xyz="${x_reflect * 0.115} ${y_reflect * 0.115} -0.015" rpy="0 0 0"/>
+      <origin xyz="${x_reflect * 0.115} ${y_reflect * 0.140} -0.015" rpy="0 0 0"/>
       <axis xyz="0 1 0"/>
     </joint>

File: urdf/robot.urdf.xacro (robot description, xacro)
@@ -204,5 +204,5 @@
   </joint>
   <!-- ========================================================================= -->
-  <!-- WHEELS (Radius = 0.045m, Width = 0.03m)                                   -->
+  <!-- WHEELS (Radius = 0.050m, Width = 0.03m, Base = 0.28m)                                   -->
   <!-- ========================================================================= -->
   <xacro:macro name="wheel" params="prefix x_reflect y_reflect">
@@ -211,5 +211,5 @@
         <origin xyz="0 0 0" rpy="${pi/2} 0 0"/>
         <geometry>
-          <cylinder radius="0.045" length="0.03"/>
+          <cylinder radius="0.050" length="0.03"/>
         </geometry>
         <material name="black"/>
@@ -218,5 +218,5 @@
         <origin xyz="0 0 0" rpy="${pi/2} 0 0"/>
         <geometry>
-          <cylinder radius="0.045" length="0.03"/>
+          <cylinder radius="0.050" length="0.03"/>
         </geometry>
       </collision>
@@ -224,5 +224,5 @@
         <origin xyz="0 0 0" rpy="${pi/2} 0 0"/>
         <mass value="0.1"/>
-        <inertia ixx="0.000058" ixy="0.0" ixz="0.0" iyy="0.000058" iyz="0.0" izz="0.000101"/>
+        <inertia ixx="0.000070" ixy="0.0" ixz="0.0" iyy="0.000070" iyz="0.0" izz="0.000125"/>
       </inertial>
     </link>
@@ -230,5 +230,5 @@
       <parent link="base_link"/>
       <child link="${prefix}_wheel"/>
-      <origin xyz="${x_reflect * 0.115} ${y_reflect * 0.115} -0.015" rpy="0 0 0"/>
+      <origin xyz="${x_reflect * 0.115} ${y_reflect * 0.140} -0.015" rpy="0 0 0"/>
       <axis xyz="0 1 0"/>
       <dynamics damping="0.01" friction="0.1"/>
@@ -253,6 +253,6 @@
       <left_joint>front_left_wheel_joint</left_joint>
       <right_joint>front_right_wheel_joint</right_joint>
-      <wheel_separation>0.768</wheel_separation>
-      <wheel_radius>0.045</wheel_radius>
+      <wheel_separation>0.28</wheel_separation>
+      <wheel_radius>0.050</wheel_radius>
       <odom_publish_frequency>30</odom_publish_frequency>
       <topic>/cmd_vel</topic>
@@ -265,6 +265,6 @@
       <left_joint>rear_left_wheel_joint</left_joint>
       <right_joint>rear_right_wheel_joint</right_joint>
-      <wheel_separation>0.768</wheel_separation>
-      <wheel_radius>0.045</wheel_radius>
+      <wheel_separation>0.28</wheel_separation>
+      <wheel_radius>0.050</wheel_radius>
       <odom_publish_frequency>0</odom_publish_frequency>
       <topic>/cmd_vel</topic>
